File: main.brd (EAGLE design)
At the start: 117.1 x 44.4 mm, 70 parts, among them CN10 PBS-8-1.27-VERTICAL, CN11 PBS-2-VERTICAL, CN12 PBS-2-VERTICAL, CN13 PBS-4-VERTICAL, CN14 PBS-2-VERTICAL, CN8 PBS-3-VERTICAL, CN9 PBS-8-1.27-VERTICAL, IC5 74LS595D, IC6 74LS595D, IC7 MC34063AD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

Commit message: Value and name were changed. Eagle is 9.2.0
Parts:
- R24: value 5.1k -> 5.6k
Other:
- board text added: "Polyakov Konstantin Russia, Yeysk, 2018-05-16, WFPS-0-1-1 Based on WFR-0-3-1"
- board text removed: "Polyakov Konstantin Russia, Yeysk, 2018-05-16, v0.3 rev1 mod1"
