File: main.sch (EAGLE design)
At the start: 70 parts, among them CN10 PBS-8-1.27-VERTICAL, CN11 PBS-2-VERTICAL, CN12 PBS-2-VERTICAL, CN13 PBS-4-VERTICAL, CN14 PBS-2-VERTICAL, CN8 PBS-3-VERTICAL, CN9 PBS-8-1.27-VERTICAL, IC5 74LS595D, IC6 74LS595D, IC7 MC34063AD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

Commit message: Value and name were changed. Eagle is 9.2.0
Parts:
- R24: value 5.1k -> 5.6k
